File: prod/atma.kicad_pcb (KiCad board)
At the start: 2 copper layers, 114.1 x 81 mm, 23 parts

Commit message: reorganize repo
Parts:
- moved ? 38.3 mm to (246.5, 121.7)
- moved _5 19.0 mm to (237.9, 166.7)
Other:
- outline, holes or cut-outs redrawn
Changed lines of the file:
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@@
     )
     (module "44144-0003" (layer F.Cu)
-      (at 247.45000000000002 160.02 180)
+      (at 246.4975 121.7295 180)
       (fp_line (start -7.62 0) (end 7.62 0) (layer F.Fab) (width 0.2))
       (fp_line (start 7.62 0) (end 7.62 16.89) (layer F.Fab) (width 0.2))
@@
     )
     (module "MountingHole_2.2mm_M2_Pad_Via" (version 20210722) (generator pcbnew) (layer "F.Cu")
-      (at 218.925 166.6875 0)
+      (at 237.925 166.6875 0)
       (fp_text reference "_5" (at 0 -3.2) (layer "F.SilkS") hide
         (effects (font (size 1 1) (thickness 0.15)))
@@
             )
             (gr_line (start 142.875 182.7375) (end 142.875 107.77499999999999) (angle 90) (layer Edge.Cuts) (width 0.15))
-(gr_line (start 145.875 104.77499999999999) (end 245.107670775 104.77499999999999) (angle 90) (layer Edge.Cuts) (width 0.15))
-(gr_line (start 248.01809829852945 107.04739319411772) (end 256.8849966358661 142.51498654346437) (angle 90) (layer Edge.Cuts) (width 0.15))
-(gr_line (start 256.97456711245326 143.24609284946928) (end 256.9284954803149 182.74099950006348) (angle 90) (layer Edge.Cuts) (width 0.15))
-(gr_line (start 145.875 185.7375) (end 253.92849748019836 185.7375) (angle 90) (layer Edge.Cuts) (width 0.15))
+(gr_line (start 145.875 104.77499999999999) (end 253.97314674624053 104.77499999999999) (angle 90) (layer Edge.Cuts) (width 0.15))
+(gr_line (start 256.97314614617886 107.77685279992875) (end 256.92685156535435 182.73935279995203) (angle 90) (layer Edge.Cuts) (width 0.15))
+(gr_line (start 145.875 185.7375) (end 253.9268521654161 185.7375) (angle 90) (layer Edge.Cuts) (width 0.15))
 (gr_arc (start 145.875 107.77499999999999) (end 145.875 104.77499999999999) (angle -90) (layer Edge.Cuts) (width 0.15))
-(gr_arc (start 245.107670775 107.77499999999999) (end 248.018098275 107.04739319999999) (angle -75.96375792170193) (layer Edge.Cuts) (width 0.15))
-(gr_arc (start 253.97456911233672 143.24259334934675) (end 256.97456711233673 143.24609284934675) (angle -14.103077621681855) (layer Edge.Cuts) (width 0.15))
-(gr_arc (start 253.92849748019836 182.73749999998836) (end 253.92849748019836 185.73749999998836) (angle -89.93316445752373) (layer Edge.Cuts) (width 0.15))
+(gr_arc (start 253.97314674624053 107.77499999999999) (end 256.97314614624054 107.77685279999999) (angle -90.03538587464544) (layer Edge.Cuts) (width 0.15))
+(gr_arc (start 253.9268521654161 182.73749999998836) (end 253.9268521654161 185.73749999998836) (angle -89.96461412468767) (layer Edge.Cuts) (width 0.15))
 (gr_arc (start 145.875 182.7375) (end 142.875 182.7375) (angle -90) (layer Edge.Cuts) (width 0.15))
 )

Commit message: finished routing
Parts:
- added G***: LOGO, main:north-sky-silk, F.Cu at (201.0, 145.7)
- added G***: LOGO, main:north-sky-silk, B.Cu at (198.7, 146.7)
Routing:
- net 3V3: track 0.00 -> 174.5 mm, vias 0 -> 2
- net matrix_inner_top: track 0.00 -> 131.8 mm
- net GP13: track 0.00 -> 131.1 mm, vias 0 -> 1
- net GP12: track 0.00 -> 128.9 mm, vias 0 -> 1
- net thumbfan_far_home: track 0.00 -> 124.7 mm
- net matrix_index_top: track 0.00 -> 121.5 mm
- net matrix_inner_home: track 0.00 -> 115.6 mm
- net thumbfan_home_home: track 0.00 -> 106.8 mm
- net matrix_index_home: track 0.00 -> 102.1 mm
- net matrix_inner_bottom: track 0.00 -> 98.8 mm
- net matrix_ring_top: track 0.00 -> 89.5 mm
- net thumbfan_near_home: track 0.00 -> 83.8 mm
- net matrix_middle_top: track 0.00 -> 82.1 mm
- net matrix_index_bottom: track 0.00 -> 81.7 mm
- net matrix_ring_home: track 0.00 -> 70.7 mm
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- added copper zone on B.Cu, net GND
- added copper zone on F.Cu, net GND
Other:
- net class Default removed
